File: zipitbreakout.sch (KiCad schematic (older format))
At the start: 3 parts, among them J1 USB_2, P1 DIL38, P2 ST60X-36S

Commit message: Finish design, first cut of board layout for prototyping
Parts:
- removed J1: USB_2, symbol USB_2
- removed P1: DIL38, symbol DIL38
- added C1: 3.3uF, ~, symbol C
- added C2: 4.7uF, ~, symbol C
- added JP1, JP2: JUMPER, ~, symbol JUMPER
- added K1: CONN_3, ~, symbol CONN_3
- added L1: 1 uH, ~, symbol INDUCTOR
- added P2: CONN_5, ~, symbol CONN_5
- added P3: CONN_4, ~, symbol CONN_4
- added P4: CONN_3X2, ~, symbol CONN_3X2
- added P5: CONN_9X2, ~, symbol CONN_9X2
- added REG1: TPS61240, symbol TPS61240
- added USB1, USB2: USB, ~, symbol USB
- P1: renamed from P2; value ST60X-36S -> Z2DOCK; symbol ST60X-36S -> Z2DOCK
Connections:
- net labels added: 1V8, 3V3, ADC_IN, AUDIO_COMMON, BTRXD_GP42, CAM_D0_GP81, CAM_D1_GP114, CAM_D2_GP51, CAM_D3_GP50, CAM_D4_GP52, CAM_D5_GP94, CAM_D6_GP93, CAM_D7_GP12, CAM_FV_GP84, CAM_LV_GP44, CAM_MCLK_GP53, CAM_PCLK_GP54, DC_IN, GP45, I2C_SCL, I2C_SDA, MIC_IN, REG_5V, SSPRXD2_GP86, USBD+, USBD-, USB_DEVICE_POWER, USB_VCC
- net labels removed: VCC, Z2-1, Z2-16, Z2-17, Z2-18, Z2-2, Z2-20, Z2-21, Z2-23, Z2-24, Z2-25, Z2-26, Z2-27, Z2-28, Z2-29, Z2-3, Z2-30, Z2-31, Z2-32, Z2-33, Z2-34, Z2-35, Z2-36, Z2-4, Z2-5, Z2-6, Z2-7, Z2-GND, Z2-USBD+, Z2-USBD-, Z2-VCC
- wire segments 80 -> 111
- no-connect marks 2 -> 3
Other:
- note added: "Camera"
- note added: "Jumpers to detach USB-B from USB-A\n(allows connecting a USB charger & a USB device)"
- note added: "Misc IO\n\n"
- note added: "Power"
- note added: "USB A Socket (host mode)"
- note added: "USB B Socket (device mode)"
- note added: "USB Battery Power - 3.3V to 5V Boost Converter (approx 350mA output)"
- note added: "USB Host Power Selector (Ext In Only or Battery)"
- note added: "i2c"
