File: z2breakout.sch (KiCad schematic (older format))
At the start: 14 parts, among them K1 CONN_3, P1 Z2DOCK, P2 CONN_5, P3 CONN_4, P4 CONN_3X2, P5 CONN_9X2

Commit message: Reroute with correct pin order, better connector spacing
Parts:
- removed P2: CONN_5, ~, symbol CONN_5
- removed P3: CONN_4, ~, symbol CONN_4
- added P2: CONN_8, symbol CONN_8
- K1: footprint ~ -> (none)
Connections:
- wire segments 111 -> 108
Other:
- note added: "Jumper USB host power from either onboard reg or DC In"
- note added: "i2c + Misc"
- note removed: "Misc IO\n\n"
- note removed: "USB Host Power Selector (Ext In Only or Battery)"
- note removed: "i2c"
- moved on the sheet: C1, C2, JP1, JP2, L1, P1, REG1, USB1, USB2

Commit message: Clean up silkscreen a bit, add i2c pullup resistors
Parts:
- added R1, R2: 10K, ~, symbol R
Connections:
- wire segments 108 -> 111
